Commit message: Add RViz configuration and update launch files for simulation
- Introduced a new RViz configuration file for better visualization.
- Updated launch files to include an option to start RViz with the simulation.
- Changed base frame ID from `base_link` to `base_footprint` in controller configurations.
- Added necessary dependencies for RViz in package.xml.

File: bunker_sim/bunker_description/urdf/bunker.xacro (robot description, xacro)
@@ -1029,4 +1029,29 @@
         <param name="max">20</param>
       </command_interface>
+      <state_interface name="position"/>
+      <state_interface name="velocity"/>
+    </joint>
+    <!-- Passive track wheels need state interfaces so robot_state_publisher can publish TF. -->
+    <joint name="wheel1.1_joint">
+      <state_interface name="position"/>
+      <state_interface name="velocity"/>
+    </joint>
+    <joint name="wheel1.3_joint">
+      <state_interface name="position"/>
+      <state_interface name="velocity"/>
+    </joint>
+    <joint name="wheel2.1_joint">
+      <state_interface name="position"/>
+      <state_interface name="velocity"/>
+    </joint>
+    <joint name="wheel2.3_joint">
+      <state_interface name="position"/>
+      <state_interface name="velocity"/>
+    </joint>
+    <joint name="wheel3.3_joint">
+      <state_interface name="position"/>
+      <state_interface name="velocity"/>
+    </joint>
+    <joint name="wheel4.3_joint">
       <state_interface name="position"/>
       <state_interface name="velocity"/>

File: bunker_sim/bunker_description/urdf/bunkeranka.xacro (robot description, xacro)
@@ -1052,4 +1052,29 @@
         <param name="max">20</param>
       </command_interface>
+      <state_interface name="position"/>
+      <state_interface name="velocity"/>
+    </joint>
+    <!-- Passive track wheels need state interfaces so robot_state_publisher can publish TF. -->
+    <joint name="wheel1.1_joint">
+      <state_interface name="position"/>
+      <state_interface name="velocity"/>
+    </joint>
+    <joint name="wheel1.3_joint">
+      <state_interface name="position"/>
+      <state_interface name="velocity"/>
+    </joint>
+    <joint name="wheel2.1_joint">
+      <state_interface name="position"/>
+      <state_interface name="velocity"/>
+    </joint>
+    <joint name="wheel2.3_joint">
+      <state_interface name="position"/>
+      <state_interface name="velocity"/>
+    </joint>
+    <joint name="wheel3.3_joint">
+      <state_interface name="position"/>
+      <state_interface name="velocity"/>
+    </joint>
+    <joint name="wheel4.3_joint">
       <state_interface name="position"/>
       <state_interface name="velocity"/>

File: bunker_sim/bunker_description/urdf/bunkur.xacro (robot description, xacro)
@@ -1054,4 +1054,29 @@
         <param name="max">20</param>
       </command_interface>
+      <state_interface name="position"/>
+      <state_interface name="velocity"/>
+    </joint>
+    <!-- Passive track wheels need state interfaces so robot_state_publisher can publish TF. -->
+    <joint name="wheel1.1_joint">
+      <state_interface name="position"/>
+      <state_interface name="velocity"/>
+    </joint>
+    <joint name="wheel1.3_joint">
+      <state_interface name="position"/>
+      <state_interface name="velocity"/>
+    </joint>
+    <joint name="wheel2.1_joint">
+      <state_interface name="position"/>
+      <state_interface name="velocity"/>
+    </joint>
+    <joint name="wheel2.3_joint">
+      <state_interface name="position"/>
+      <state_interface name="velocity"/>
+    </joint>
+    <joint name="wheel3.3_joint">
+      <state_interface name="position"/>
+      <state_interface name="velocity"/>
+    </joint>
+    <joint name="wheel4.3_joint">
       <state_interface name="position"/>
       <state_interface name="velocity"/>
