Commit message: Add initial joint configuration parameters for UR robot in launch files

File: bunker_sim/bunker_description/urdf/bunkur.xacro (robot description, xacro)
@@ -20,8 +20,22 @@
   <xacro:arg name="ur_mount_xyz" default="0.3 0 0.05"/>
   <xacro:arg name="ur_mount_rpy" default="0 0 0"/>
+  <xacro:arg name="ur_initial_shoulder_pan_joint" default="0.1745329252"/>
+  <xacro:arg name="ur_initial_shoulder_lift_joint" default="-1.57"/>
+  <xacro:arg name="ur_initial_elbow_joint" default="1.5707963268"/>
+  <xacro:arg name="ur_initial_wrist_1_joint" default="-1.57"/>
+  <xacro:arg name="ur_initial_wrist_2_joint" default="-1.5707963268"/>
+  <xacro:arg name="ur_initial_wrist_3_joint" default="0.0"/>
   <xacro:arg name="ur_joint_limit_params" default="$(find ur_description)/config/$(arg ur_type)/joint_limits.yaml"/>
   <xacro:arg name="ur_kinematics_params" default="$(find ur_description)/config/$(arg ur_type)/default_kinematics.yaml"/>
   <xacro:arg name="ur_physical_params" default="$(find ur_description)/config/$(arg ur_type)/physical_parameters.yaml"/>
   <xacro:arg name="ur_visual_params" default="$(find ur_description)/config/$(arg ur_type)/visual_parameters.yaml"/>
+  <xacro:property name="ur_initial_positions" value="${dict(
+      shoulder_pan_joint=float('$(arg ur_initial_shoulder_pan_joint)'),
+      shoulder_lift_joint=float('$(arg ur_initial_shoulder_lift_joint)'),
+      elbow_joint=float('$(arg ur_initial_elbow_joint)'),
+      wrist_1_joint=float('$(arg ur_initial_wrist_1_joint)'),
+      wrist_2_joint=float('$(arg ur_initial_wrist_2_joint)'),
+      wrist_3_joint=float('$(arg ur_initial_wrist_3_joint)')
+    )}"/>
   <xacro:ur_robot
       name="$(arg ur_type)"
@@ -37,5 +51,6 @@
   <xacro:ur_ros2_control
       name="URSimSystem"
-      tf_prefix="$(arg ur_tf_prefix)"/>
+      tf_prefix="$(arg ur_tf_prefix)"
+      initial_positions="${ur_initial_positions}"/>
   <link
     name="base_link">

Commit message: made bunker using tracked system in gz sim

File: bunker_sim/bunker_description/urdf/bunkur.xacro (robot description, xacro)
@@ -6,4 +6,5 @@
   <!-- xacro arg for controller params file (absolute path) injected from launch -->
   <xacro:arg name="controllers_yaml" default=""/>
+  <xacro:arg name="tracked_cmd_topic" default="/bunker/tracked_cmd_vel"/>
   <!-- KDL requires the root link to have no inertia. -->
   <link name="base_footprint"/>
@@ -93,4 +94,52 @@
     </collision>
   </link>
+  <!--
+    Gazebo's native tracked-vehicle systems act on collision links representing
+    each continuous track. The visible wheel links remain for the model and arm
+    kinematics, but their contacts are frictionless below so they do not fight
+    the commanded track surface velocity during skid steering.
+  -->
+  <link name="left_track">
+    <inertial>
+      <origin xyz="0 0 0"/>
+      <mass value="1.0"/>
+      <inertia ixx="0.01" ixy="0" ixz="0" iyy="0.08" iyz="0" izz="0.08"/>
+    </inertial>
+    <collision>
+      <origin xyz="0 0 0"/>
+      <geometry>
+        <box size="0.90 0.11 0.064"/>
+      </geometry>
+    </collision>
+  </link>
+  <joint name="left_track_joint" type="fixed">
+    <parent link="base_link"/>
+    <child link="left_track"/>
+    <origin xyz="0.0275 0.3495 -0.326"/>
+  </joint>
+  <link name="right_track">
+    <inertial>
+      <origin xyz="0 0 0"/>
+      <mass value="1.0"/>
+      <inertia ixx="0.01" ixy="0" ixz="0" iyy="0.08" iyz="0" izz="0.08"/>
+    </inertial>
+    <collision>
+      <origin xyz="0 0 0"/>
+      <geometry>
+        <box size="0.90 0.11 0.064"/>
+      </geometry>
+    </collision>
+  </link>
+  <joint name="right_track_joint" type="fixed">
+    <parent link="base_link"/>
+    <child link="right_track"/>
+    <origin xyz="0.0275 -0.3495 -0.326"/>
+  </joint>
+  <gazebo reference="left_track_joint">
+    <preserveFixedJoint>true</preserveFixedJoint>
+  </gazebo>
+  <gazebo reference="right_track_joint">
+    <preserveFixedJoint>true</preserveFixedJoint>
+  </gazebo>
   <link
     name="wheel1_Link">
@@ -1109,47 +1158,113 @@
     </plugin>
   </gazebo>
-  <!-- Gazebo physics tuning: ensure wheel collisions have enough friction so
-       wheel rotation turns into traction (otherwise the wheels can spin in place).
-       Adjust mu1/mu2 if it still slips. -->
+  <gazebo>
+    <plugin
+      filename="gz-sim-tracked-vehicle-system"
+      name="gz::sim::systems::TrackedVehicle">
+      <left_track>
+        <link>left_track</link>
+      </left_track>
+      <right_track>
+        <link>right_track</link>
+      </right_track>
+      <tracks_separation>0.699</tracks_separation>
+      <tracks_height>0.064</tracks_height>
+      <steering_efficiency>1.0</steering_efficiency>
+      <topic>$(arg tracked_cmd_topic)</topic>
+      <odom_topic>/odom</odom_topic>
+      <odom_publish_frequency>50</odom_publish_frequency>
+    </plugin>
+    <plugin
+      filename="gz-sim-track-controller-system"
+      name="gz::sim::systems::TrackController">
+      <link>left_track</link>
+      <min_velocity>-1.0</min_velocity>
+      <max_velocity>1.0</max_velocity>
+    </plugin>
+    <plugin
+      filename="gz-sim-track-controller-system"
+      name="gz::sim::systems::TrackController">
+      <link>right_track</link>
+      <min_velocity>-1.0</min_velocity>
+      <max_velocity>1.0</max_velocity>
+    </plugin>
+  </gazebo>
+  <gazebo reference="left_track">
+    <mu1>0.7</mu1>
+    <mu2>150.0</mu2>
+    <fdir1>0 1 0</fdir1>
+    <maxContacts>20</maxContacts>
+  </gazebo>
+  <gazebo reference="right_track">
+    <mu1>0.7</mu1>
+    <mu2>150.0</mu2>
+    <fdir1>0 1 0</fdir1>
+    <maxContacts>20</maxContacts>
+  </gazebo>
+  <!-- The native track links provide traction. Wheel contacts are visual/support
+       geometry only and must not oppose lateral skid during an in-place turn. -->
   <gazebo reference="wheel1_Link">
-    <mu1>0.8</mu1>
-    <mu2>0.8</mu2>
+    <mu1>0.0</mu1>
+    <mu2>0.0</mu2>
   </gazebo>
   <gazebo reference="wheel2_Link">
-    <mu1>0.8</mu1>
-    <mu2>0.8</mu2>
+    <mu1>0.0</mu1>
+    <mu2>0.0</mu2>
   </gazebo>
   <gazebo reference="wheel3_Link">
-    <mu1>0.8</mu1>
-    <mu2>0.8</mu2>
+    <mu1>0.0</mu1>
+    <mu2>0.0</mu2>
   </gazebo>
   <gazebo reference="wheel4_Link">
-    <mu1>0.8</mu1>
-    <mu2>0.8</mu2>
-  </gazebo>
-  <!-- Friction parameters for additional track wheels -->
+    <mu1>0.0</mu1>
+    <mu2>0.0</mu2>
+  </gazebo>
   <gazebo reference="wheel1.2_Link">
-    <mu1>0.8</mu1>
-    <mu2>0.8</mu2>
+    <mu1>0.0</mu1>
+    <mu2>0.0</mu2>
+  </gazebo>
+  <gazebo reference="wheel1.1_Link">
+    <mu1>0.0</mu1>
+    <mu2>0.0</mu2>
+  </gazebo>
+  <gazebo reference="wheel1.3_Link">
+    <mu1>0.0</mu1>
+    <mu2>0.0</mu2>
+  </gazebo>
+  <gazebo reference="wheel2.1_Link">
+    <mu1>0.0</mu1>
+    <mu2>0.0</mu2>
+  </gazebo>
+  <gazebo reference="wheel2.3_Link">
+    <mu1>0.0</mu1>
+    <mu2>0.0</mu2>
   </gazebo>
   <gazebo reference="wheel3.1_Link">
-    <mu1>0.8</mu1>
-    <mu2>0.8</mu2>
+    <mu1>0.0</mu1>
+    <mu2>0.0</mu2>
   </gazebo>
   <gazebo reference="wheel3.2_Link">
-    <mu1>0.8</mu1>
-    <mu2>0.8</mu2>
+    <mu1>0.0</mu1>
+    <mu2>0.0</mu2>
   </gazebo>
   <gazebo reference="wheel4.1_Link">
-    <mu1>0.8</mu1>
-    <mu2>0.8</mu2>
+    <mu1>0.0</mu1>
+    <mu2>0.0</mu2>
   </gazebo>
   <gazebo reference="wheel4.2_Link">
-    <mu1>0.8</mu1>
-    <mu2>0.8</mu2>
+    <mu1>0.0</mu1>
+    <mu2>0.0</mu2>
+  </gazebo>
+  <gazebo reference="wheel3.3_Link">
+    <mu1>0.0</mu1>
+    <mu2>0.0</mu2>
+  </gazebo>
+  <gazebo reference="wheel4.3_Link">
+    <mu1>0.0</mu1>
+    <mu2>0.0</mu2>
   </gazebo>
   <gazebo reference="wheel2.2_Link">
-    <mu1>0.8</mu1>
-    <mu2>0.8</mu2>
+    <mu1>0.0</mu1>
+    <mu2>0.0</mu2>
   </gazebo>
 </robot>
