Commit message: Update RB-VOGUI configuration for UR20 arm and add lift position controller

File: rbvogui_ur_sim_setup/urdf/rbvogui_ur_standard_control.urdf.xacro (robot description, xacro)
@@ -8,9 +8,11 @@
     filename="$(find robotnik_description)/urdf/wheels/steering_wheel/steering_wheel.urdf.xacro" />
   <xacro:include
+    filename="$(find robotnik_description)/urdf/structures/ewellix/all_ewellix_lift.urdf.xacro" />
+  <xacro:include
     filename="$(find robotnik_description)/urdf/arms/ur_macro.urdf.xacro" />
   <xacro:arg name="namespace" default="robot" />
   <xacro:arg name="prefix" default="robot_" />
   <xacro:arg name="gazebo_ignition" default="true" />
-  <xacro:arg name="ur_type" default="ur5e" />
+  <xacro:arg name="ur_type" default="ur20" />
   <xacro:property name="wheel_offset_x" value="0.368" />
   <xacro:property name="wheel_offset_y" value="0.235" />
@@ -44,10 +46,16 @@
     <origin xyz="-${wheel_offset_x} -${wheel_offset_y} 0" rpy="0 0 0" />
   </xacro:steering_wheel>
+  <xacro:ewellix_lift_900mm
+    prefix="$(arg prefix)lift_"
+    parent="$(arg prefix)chassis_link"
+    cut_model="true">
+    <origin xyz="0 0 0.235" rpy="0 0 0" />
+  </xacro:ewellix_lift_900mm>
   <xacro:arm_ur
     ur_type="$(arg ur_type)"
     frame_prefix="$(arg prefix)arm_"
-    parent="$(arg prefix)chassis_link"
+    parent="$(arg prefix)lift_top_link"
     gazebo_ignition="$(arg gazebo_ignition)">
-    <origin xyz="0 0 0.235" rpy="0 0 0" />
+    <origin xyz="0 0 0" rpy="0 0 0" />
   </xacro:arm_ur>
   <xacro:if value="$(arg gazebo_ignition)">

Commit message: Update RB-VOGUI-XL configuration and add lift position controller for simulation

File: rbvogui_ur_sim_setup/urdf/rbvogui_ur_standard_control.urdf.xacro (robot description, xacro)
@@ -4,9 +4,7 @@
     filename="$(find robotnik_description)/urdf/inertia.urdf.xacro" />
   <xacro:include
-    filename="$(find robotnik_description)/urdf/bodies/rbvogui/rbvogui_body.urdf.xacro" />
+    filename="$(find robotnik_description)/urdf/bodies/rbvogui_xl/rbvogui_xl_body.urdf.xacro" />
   <xacro:include
-    filename="$(find robotnik_description)/urdf/wheels/steering_wheel/steering_wheel.urdf.xacro" />
-  <xacro:include
-    filename="$(find robotnik_description)/urdf/structures/ewellix/all_ewellix_lift.urdf.xacro" />
+    filename="$(find robotnik_description)/urdf/wheels/steering_wheel/steering_wheel_285.urdf.xacro" />
   <xacro:include
     filename="$(find robotnik_description)/urdf/arms/ur_macro.urdf.xacro" />
@@ -15,8 +13,8 @@
   <xacro:arg name="gazebo_ignition" default="true" />
   <xacro:arg name="ur_type" default="ur20" />
-  <xacro:property name="wheel_offset_x" value="0.368" />
-  <xacro:property name="wheel_offset_y" value="0.235" />
-  <xacro:rbvogui_body prefix="$(arg prefix)" hq="true" />
-  <xacro:steering_wheel
+  <xacro:property name="wheel_offset_x" value="0.4795" />
+  <xacro:property name="wheel_offset_y" value="0.2925" />
+  <xacro:rbvogui_xl_body prefix="$(arg prefix)" hq="true" />
+  <xacro:steering_xl_wheel_285
     prefix="$(arg prefix)front_right_"
     parent="$(arg prefix)base_link"
@@ -24,6 +22,6 @@
     hq="true">
     <origin xyz="${wheel_offset_x} -${wheel_offset_y} 0" rpy="0 0 0" />
-  </xacro:steering_wheel>
-  <xacro:steering_wheel
+  </xacro:steering_xl_wheel_285>
+  <xacro:steering_xl_wheel_285
     prefix="$(arg prefix)front_left_"
     parent="$(arg prefix)base_link"
@@ -31,6 +29,6 @@
     hq="true">
     <origin xyz="${wheel_offset_x} ${wheel_offset_y} 0" rpy="0 0 0" />
-  </xacro:steering_wheel>
-  <xacro:steering_wheel
+  </xacro:steering_xl_wheel_285>
+  <xacro:steering_xl_wheel_285
     prefix="$(arg prefix)back_left_"
     parent="$(arg prefix)base_link"
@@ -38,6 +36,6 @@
     hq="true">
     <origin xyz="-${wheel_offset_x} ${wheel_offset_y} 0" rpy="0 0 0" />
-  </xacro:steering_wheel>
-  <xacro:steering_wheel
+  </xacro:steering_xl_wheel_285>
+  <xacro:steering_xl_wheel_285
     prefix="$(arg prefix)back_right_"
     parent="$(arg prefix)base_link"
@@ -45,15 +43,74 @@
     hq="true">
     <origin xyz="-${wheel_offset_x} -${wheel_offset_y} 0" rpy="0 0 0" />
-  </xacro:steering_wheel>
-  <xacro:ewellix_lift_900mm
-    prefix="$(arg prefix)lift_"
-    parent="$(arg prefix)chassis_link"
-    cut_model="true">
-    <origin xyz="0 0 0.235" rpy="0 0 0" />
-  </xacro:ewellix_lift_900mm>
+  </xacro:steering_xl_wheel_285>
+  <link name="$(arg prefix)lift_base_link">
+    <visual>
+      <geometry>
+        <mesh
+          filename="package://robotnik_description/meshes/structures/ewellix/ewellix_lift_base_900mm.stl"
+          scale="0.95 0.95 1" />
+      </geometry>
+      <material name="grey">
+        <color rgba="0.7 0.7 0.7 1" />
+      </material>
+    </visual>
+    <collision>
+      <origin xyz="-0.005 0 0.00235" rpy="0 0 0" />
+      <geometry>
+        <mesh
+          filename="package://robotnik_description/meshes/structures/ewellix/ewellix_lift_base_900mm.stl"
+          scale="0.95 0.95 1" />
+      </geometry>
+    </collision>
+    <inertial>
+      <mass value="20" />
+      <origin xyz="0 0 0" rpy="0 0 0" />
+      <inertia ixx="1e-1" ixy="0" ixz="0" iyy="1e-1" iyz="0" izz="1e-1" />
+    </inertial>
+  </link>
+  <joint name="$(arg prefix)lift_base_joint" type="fixed">
+    <origin xyz="0.26 0 0.01" rpy="0 0 0" />
+    <parent link="$(arg prefix)chassis_link" />
+    <child link="$(arg prefix)lift_base_link" />
+  </joint>
+  <link name="$(arg prefix)lift_link">
+    <visual>
+      <geometry>
+        <mesh filename="package://robotnik_description/meshes/structures/ewellix/ewellix_lift_top_900mm.stl" />
+      </geometry>
+      <material name="grey">
+        <color rgba="0.7 0.7 0.7 1" />
+      </material>
+    </visual>
+    <collision>
+      <origin xyz="-0.005 0 0.00235" rpy="0 0 0" />
+      <geometry>
+        <mesh filename="package://robotnik_description/meshes/structures/ewellix/ewellix_lift_top_900mm.stl" />
+      </geometry>
+    </collision>
+    <inertial>
+      <mass value="2" />
+      <origin xyz="0 0 0" rpy="0 0 0" />
+      <inertia ixx="0.02" ixy="0" ixz="0" iyy="0.02" iyz="0" izz="0.02" />
+    </inertial>
+  </link>
+  <joint name="$(arg prefix)lift_joint" type="prismatic">
+    <origin xyz="0 0 0" rpy="0 0 0" />
+    <parent link="$(arg prefix)lift_base_link" />
+    <child link="$(arg prefix)lift_link" />
+    <limit effort="1000" lower="0.0" upper="0.9" velocity="0.088" />
+    <axis xyz="0 0 1" />
+    <dynamics damping="0.0" friction="0.0" />
+  </joint>
+  <gazebo reference="$(arg prefix)lift_base_link">
+    <material>Gazebo/Grey</material>
+  </gazebo>
+  <gazebo reference="$(arg prefix)lift_link">
+    <material>Gazebo/Grey</material>
+  </gazebo>
   <xacro:arm_ur
     ur_type="$(arg ur_type)"
     frame_prefix="$(arg prefix)arm_"
-    parent="$(arg prefix)lift_top_link"
+    parent="$(arg prefix)lift_link"
     gazebo_ignition="$(arg gazebo_ignition)">
     <origin xyz="0 0 0" rpy="0 0 0" />
@@ -119,4 +176,7 @@
         name="$(arg prefix)back_right_wheel_joint"
         command_interface="velocity" lower_limit="-10.0" upper_limit="10.0" />
+      <xacro:controlled_joint
+        name="$(arg prefix)lift_joint"
+        command_interface="position" lower_limit="0.0" upper_limit="0.9" />
     </ros2_control>
   </xacro:if>

Commit message: Update README and URDF files: adjust lift initial position and add lift height properties

File: rbvogui_ur_sim_setup/urdf/rbvogui_ur_standard_control.urdf.xacro (robot description, xacro)
@@ -15,4 +15,10 @@
   <xacro:property name="wheel_offset_x" value="0.4795" />
   <xacro:property name="wheel_offset_y" value="0.2925" />
+  <xacro:property name="chassis_top_plate_z" value="0.2879" />
+  <xacro:property name="lift_base_mount_z" value="0.01" />
+  <xacro:property name="lift_retracted_height_above_top_plate" value="0.35" />
+  <xacro:property
+    name="lift_retracted_origin_z"
+    value="${chassis_top_plate_z - lift_base_mount_z + lift_retracted_height_above_top_plate}" />
   <xacro:rbvogui_xl_body prefix="$(arg prefix)" hq="true" />
   <xacro:steering_xl_wheel_285
@@ -70,5 +76,5 @@
   </link>
   <joint name="$(arg prefix)lift_base_joint" type="fixed">
-    <origin xyz="0.26 0 0.01" rpy="0 0 0" />
+    <origin xyz="0.26 0 ${lift_base_mount_z}" rpy="0 0 0" />
     <parent link="$(arg prefix)chassis_link" />
     <child link="$(arg prefix)lift_base_link" />
@@ -96,5 +102,5 @@
   </link>
   <joint name="$(arg prefix)lift_joint" type="prismatic">
-    <origin xyz="0 0 0" rpy="0 0 0" />
+    <origin xyz="0 0 ${lift_retracted_origin_z}" rpy="0 0 0" />
     <parent link="$(arg prefix)lift_base_link" />
     <child link="$(arg prefix)lift_link" />

File: rbvogui_ur_sim_setup/urdf/wheels/rubber_wheel/rubber_wheel_285.urdf.xacro (robot description, xacro)
@@ -48,32 +48,12 @@
     <link name="${prefix}wheel">
       <visual>
-        <!-- HIGH RESOLUTION WHEELS -->
-        <xacro:if value="${hq}">
-          <xacro:unless value="${reflect}">
-            <origin
-              xyz="0 0 0"
-              rpy="0 0 ${pi}" />
-          </xacro:unless>
-          <xacro:if value="${reflect}">
-            <origin
-              xyz="0 0 0"
-              rpy="0 0 0" />
-          </xacro:if>
-          <geometry>
-            <mesh
-              filename="package://rbvogui_ur_sim_setup/meshes/wheels/rubber_wheel/rubber_wheel_285.stl" />
-          </geometry>
-        </xacro:if>
-        <!-- LOW RESOLUTION WHEELS -->
-        <xacro:unless value="${hq}">
-          <origin
-            xyz="0 0 0"
-            rpy="${pi/2} 0 0" />
-          <geometry>
-            <cylinder
-              length="${rubber_wheel_width}"
-              radius="${rubber_wheel_radius}" />
-          </geometry>
-        </xacro:unless>
+        <origin
+          xyz="0 0 0"
+          rpy="${pi/2} 0 0" />
+        <geometry>
+          <cylinder
+            length="${rubber_wheel_width}"
+            radius="${rubber_wheel_radius}" />
+        </geometry>
         <material name="black">
           <color rgba="0.1 0.1 0.1 1" />

Commit message: Add initial joint positions for UR robot in URDF configuration

File: rbvogui_ur_sim_setup/urdf/rbvogui_ur_standard_control.urdf.xacro (robot description, xacro)
@@ -13,4 +13,18 @@
   <xacro:arg name="gazebo_ignition" default="true" />
   <xacro:arg name="ur_type" default="ur20" />
+  <!-- Requested pose: 180°, 90°, -90°, -90°, -90°, 0°; flange down. -->
+  <xacro:arg name="ur_initial_shoulder_pan_joint" default="3.141592653589793" />
+  <xacro:arg name="ur_initial_shoulder_lift_joint" default="3.141592653589793" />
+  <xacro:arg name="ur_initial_elbow_joint" default="-1.570796326794897" />
+  <xacro:arg name="ur_initial_wrist_1_joint" default="0.0" />
+  <xacro:arg name="ur_initial_wrist_2_joint" default="1.570796326794897" />
+  <xacro:arg name="ur_initial_wrist_3_joint" default="0.0" />
+  <xacro:property name="ur_initial_positions" value="${dict(
+    shoulder_pan_joint=float('$(arg ur_initial_shoulder_pan_joint)'),
+    shoulder_lift_joint=float('$(arg ur_initial_shoulder_lift_joint)'),
+    elbow_joint=float('$(arg ur_initial_elbow_joint)'),
+    wrist_1_joint=float('$(arg ur_initial_wrist_1_joint)'),
+    wrist_2_joint=float('$(arg ur_initial_wrist_2_joint)'),
+    wrist_3_joint=float('$(arg ur_initial_wrist_3_joint)'))}" />
   <xacro:property name="wheel_offset_x" value="0.4795" />
   <xacro:property name="wheel_offset_y" value="0.2925" />
@@ -119,5 +133,6 @@
     frame_prefix="$(arg prefix)arm_"
     parent="$(arg prefix)lift_link"
-    gazebo_ignition="$(arg gazebo_ignition)">
+    gazebo_ignition="$(arg gazebo_ignition)"
+    initial_positions="${ur_initial_positions}">
     <origin xyz="0 0 0" rpy="0 0 0" />
   </xacro:arm_ur>
